File: bottom/bottom.kicad_pcb (KiCad board)
At the start: 2 copper layers, 276.2 x 78.9 mm, 6 parts

Commit message: add mounting holes to sch
Parts:
- removed the H3 at (165.1, 113.0)
- added H4: MountingHole, MountingHole:MountingHole_2.2mm_M2_Pad, F.Cu at (254.8, 109.1)
- H1: moved to F.Cu
- H2, H5, H6: value MountingHole_2.2mm_M2_Pad -> MountingHole; moved to F.Cu
- H3: renamed from H4; value MountingHole_2.2mm_M2_Pad -> MountingHole; moved to F.Cu
- moved H5 242.6 mm to (331.2, 88.7), turned to 0 degrees
- moved H6 242.6 mm to (331.2, 146.7), turned to 0 degrees
- moved H1 234.2 mm to (92.9, 88.9), turned to 0 degrees
- moved H2 233.9 mm to (93.0, 146.8), turned to 0 degrees
- moved H3 53.2 mm to (183.4, 118.8), turned to 0 degrees
Other:
- outline, holes or cut-outs redrawn

Commit message: 3mm outer spacing
Parts:
- moved H1 245.3 mm to (338.1, 93.7)
- moved H2 245.1 mm to (338.0, 151.5)
- moved H5 231.5 mm to (99.8, 93.5)
- moved H6 231.5 mm to (99.8, 151.4)
- moved H4 78.7 mm to (176.2, 113.8)
- moved H3 64.3 mm to (247.6, 123.6)
Other:
- board size 276.2 x 78.9 mm -> 277 x 77.4 mm

Commit message: gnd zone fill
Parts:
- moved H4 19.2 mm to (157.5, 117.9)
- moved H2 18.9 mm to (324.1, 138.7)
- moved H6 15.5 mm to (90.9, 138.7)
- moved H1 14.2 mm to (324.1, 95.5)
- moved H5 9.05 mm to (90.9, 95.5)
- moved H3 7.71 mm to (252.7, 117.9)
Other:
- board size 277 x 77.4 mm -> 272.3 x 77.6 mm
Changed lines of the file:
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@@
   (general
     (thickness 1.6)
-    (drawings 12)
+    (drawings 14)
     (tracks 0)
     (zones 0)
@@
   )
   (module MountingHole:MountingHole_2.2mm_M2_Pad (layer F.Cu)
-    (at 99.7585 151.41575)
+    (at 324.104 138.684)
+    (descr "Mounting Hole 2.2mm, M2")
+    (tags "mounting hole 2.2mm m2")
+    (attr virtual)
+    (fp_text reference H2 (at 0 -3.2) (layer F.SilkS)
+      (effects (font (size 1 1) (thickness 0.15)))
+    )
+    (fp_text value MountingHole (at 0 3.2) (layer F.Fab)
+      (effects (font (size 1 1) (thickness 0.15)))
+    )
+    (fp_circle (center 0 0) (end 2.2 0) (layer Cmts.User) (width 0.15))
+    (fp_circle (center 0 0) (end 2.45 0) (layer F.CrtYd) (width 0.05))
+    (fp_text user %R (at 0.3 0) (layer F.Fab)
+      (effects (font (size 1 1) (thickness 0.15)))
+    )
+    (pad 1 thru_hole circle (at 0 0) (size 4.4 4.4) (drill 2.2) (layers *.Cu *.Mask))
+  )
+  (module MountingHole:MountingHole_2.2mm_M2_Pad (layer F.Cu)
+    (at 90.932 138.684)
     (descr "Mounting Hole 2.2mm, M2")
     (tags "mounting hole 2.2mm m2")
@@
   )
   (module MountingHole:MountingHole_2.2mm_M2_Pad (layer F.Cu)
-    (at 99.7585 93.50375)
+    (at 90.932 95.504)
     (descr "Mounting Hole 2.2mm, M2")
     (tags "mounting hole 2.2mm m2")
@@
       (effects (font (size 1 1) (thickness 0.15)))
     )
-    (fp_circle (center 0 0) (end 2.45 0) (layer F.CrtYd) (width 0.05))
-    (fp_circle (center 0 0) (end 2.2 0) (layer Cmts.User) (width 0.15))
-    (fp_text user %R (at 0.3 0) (layer F.Fab)
-      (effects (font (size 1 1) (thickness 0.15)))
-    )
-    (pad 1 thru_hole circle (at 0 0) (size 4.4 4.4) (drill 2.2) (layers *.Cu *.Mask))
-  )
-  (module MountingHole:MountingHole_2.2mm_M2_Pad (layer F.Cu)
-    (at 247.5865 123.60275)
+    (fp_circle (center 0 0) (end 2.2 0) (layer Cmts.User) (width 0.15))
+    (fp_circle (center 0 0) (end 2.45 0) (layer F.CrtYd) (width 0.05))
+    (fp_text user %R (at 0.3 0) (layer F.Fab)
+      (effects (font (size 1 1) (thickness 0.15)))
+    )
+    (pad 1 thru_hole circle (at 0 0) (size 4.4 4.4) (drill 2.2) (layers *.Cu *.Mask))
+  )
+  (module MountingHole:MountingHole_2.2mm_M2_Pad (layer F.Cu)
+    (at 252.73 117.856)
     (descr "Mounting Hole 2.2mm, M2")
     (tags "mounting hole 2.2mm m2")
@@
       (effects (font (size 1 1) (thickness 0.15)))
     )
-    (fp_circle (center 0 0) (end 2.2 0) (layer Cmts.User) (width 0.15))
-    (fp_circle (center 0 0) (end 2.45 0) (layer F.CrtYd) (width 0.05))
-    (fp_text user %R (at 0.3 0) (layer F.Fab)
-      (effects (font (size 1 1) (thickness 0.15)))
-    )
-    (pad 1 thru_hole circle (at 0 0) (size 4.4 4.4) (drill 2.2) (layers *.Cu *.Mask))
-  )
-  (module MountingHole:MountingHole_2.2mm_M2_Pad (layer F.Cu)
-    (at 176.2125 113.82375)
+    (fp_circle (center 0 0) (end 2.45 0) (layer F.CrtYd) (width 0.05))
+    (fp_circle (center 0 0) (end 2.2 0) (layer Cmts.User) (width 0.15))
+    (fp_text user %R (at 0.3 0) (layer F.Fab)
+      (effects (font (size 1 1) (thickness 0.15)))
+    )
+    (pad 1 thru_hole circle (at 0 0) (size 4.4 4.4) (drill 2.2) (layers *.Cu *.Mask))
+  )
+  (module MountingHole:MountingHole_2.2mm_M2_Pad (layer F.Cu)
+    (at 157.48 117.856)
     (descr "Mounting Hole 2.2mm, M2")
     (tags "mounting hole 2.2mm m2")
@@
   )
   (module MountingHole:MountingHole_2.2mm_M2_Pad (layer F.Cu)
-    (at 338.0105 151.54275)
-    (descr "Mounting Hole 2.2mm, M2")
-    (tags "mounting hole 2.2mm m2")
-    (attr virtual)
-    (fp_text reference H2 (at 0 -3.2) (layer F.SilkS)
-      (effects (font (size 1 1) (thickness 0.15)))
-    )
-    (fp_text value MountingHole (at 0 3.2) (layer F.Fab)
-      (effects (font (size 1 1) (thickness 0.15)))
-    )
-    (fp_circle (center 0 0) (end 2.45 0) (layer F.CrtYd) (width 0.05))
-    (fp_circle (center 0 0) (end 2.2 0) (layer Cmts.User) (width 0.15))
-    (fp_text user %R (at 0.3 0) (layer F.Fab)
-      (effects (font (size 1 1) (thickness 0.15)))
-    )
-    (pad 1 thru_hole circle (at 0 0) (size 4.4 4.4) (drill 2.2) (layers *.Cu *.Mask))
-  )
-  (module MountingHole:MountingHole_2.2mm_M2_Pad (layer F.Cu)
-    (at 338.1375 93.6625)
+    (at 324.104 95.504)
     (descr "Mounting Hole 2.2mm, M2")
     (tags "mounting hole 2.2mm m2")
@@
       (net 1 GND))
   )
-  (gr_line (start 354.584 156.7688) (end 83.566 156.7688) (layer Edge.Cuts) (width 0.05))
-  (gr_line (start 357.5812 153.7716) (end 357.5812 82.7532) (layer Edge.Cuts) (width 0.05))
-  (gr_arc (start 354.584 153.7716) (end 354.584 156.7688) (angle -90) (layer Edge.Cuts) (width 0.05))
-  (gr_line (start 333.2988 79.756) (end 83.566 79.7814) (layer Edge.Cuts) (width 0.05))
-  (gr_line (start 343.8398 79.756) (end 354.584 79.756) (layer Edge.Cuts) (width 0.05))
-  (gr_line (start 333.2988 79.756) (end 334.1116 79.4004) (layer Edge.Cuts) (width 0.05))
-  (gr_line (start 343.0524 79.4004) (end 334.1116 79.4004) (layer Edge.Cuts) (width 0.05))
-  (gr_line (start 343.8398 79.756) (end 343.0524 79.4004) (layer Edge.Cuts) (width 0.05))
-  (gr_arc (start 354.584 82.7532) (end 357.5812 82.7532) (angle -90) (layer Edge.Cuts) (width 0.05))
-  (gr_line (start 80.5688 153.7716) (end 80.5688 82.7786) (layer Edge.Cuts) (width 0.05))
-  (gr_arc (start 83.566 153.7716) (end 80.5688 153.7716) (angle -90) (layer Edge.Cuts) (width 0.05))
-  (gr_arc (start 83.566 82.7786) (end 83.566 79.7814) (angle -90) (layer Edge.Cuts) (width 0.05))
+  (gr_arc (start 340.65845 152.85085) (end 340.65845 155.84805) (angle -90) (layer Edge.Cuts) (width 0.05))
+  (gr_line (start 74.40422 78.86192) (end 318.56045 78.83525) (layer Edge.Cuts) (width 0.05))
+  (gr_line (start 74.40168 155.84678) (end 340.65845 155.84805) (layer Edge.Cuts) (width 0.05))
+  (gr_line (start 71.40194 152.84704) (end 71.41464 81.8515) (layer Edge.Cuts) (width 0.05))
+  (gr_arc (start 74.40168 152.84704) (end 71.40194 152.84704) (angle -90) (layer Edge.Cuts) (width 0.05))
+  (gr_arc (start 74.40422 81.8515) (end 74.40422 78.86192) (angle -90) (layer Edge.Cuts) (width 0.05))
+  (gr_line (start 319.19545 78.83525) (end 318.56045 78.83525) (layer Edge.Cuts) (width 0.05))
+  (gr_line (start 320.08445 78.20025) (end 319.19545 78.83525) (layer Edge.Cuts) (width 0.05))
+  (gr_line (start 329.86345 78.83525) (end 329.91425 78.83525) (layer Edge.Cuts) (width 0.05))
+  (gr_line (start 328.97445 78.20025) (end 329.86345 78.83525) (layer Edge.Cuts) (width 0.05))
+  (gr_line (start 320.08445 78.20025) (end 328.97445 78.20025) (layer Edge.Cuts) (width 0.05))
+  (gr_line (start 343.65565 152.85085) (end 343.65565 81.83245) (layer Edge.Cuts) (width 0.05))
+  (gr_line (start 329.91425 78.83525) (end 340.65845 78.83525) (layer Edge.Cuts) (width 0.05))
+  (gr_arc (start 340.65845 81.83245) (end 343.65565 81.83245) (angle -90) (layer Edge.Cuts) (width 0.05))
   (zone (net 1) (net_name GND) (layer F.Cu) (hatch edge 0.508)
     (connect_pads (clearance 0.508))
@@
     (polygon
       (pts
-        (xy 359.3592 77.3684) (xy 359.5116 161.0106) (xy 78.232 161.0106) (xy 78.232 77.343) (xy 359.3338 77.343)
+        (xy 348.45625 159.54375) (xy 69.85 159.54375) (xy 69.85 76.99375) (xy 348.45625 76.99375)
       )
     )
@@
     (polygon
       (pts
-        (xy 360.9848 76.4286) (xy 360.934 76.4286) (xy 360.9594 76.454) (xy 361.1626 76.4286) (xy 360.68 159.6136)
-        (xy 76.708 162.6362) (xy 77.4954 76.581) (xy 360.8324 76.2762)
+        (xy 348.45625 159.54375) (xy 69.85 159.54375) (xy 69.85 76.99375) (xy 348.45625 76.99375)
       )
     )

Commit message: move mounting holes and flip silk screen on pcb
Parts:
- H1, H2, H3, H4, H5, H6: moved to B.Cu
- moved H5 1.27 mm to (92.2, 95.5)
- moved H6 1.27 mm to (92.2, 138.7)
Routing:
- removed copper zone on B.Cu, net GND
- removed copper zone on F.Cu, net GND
