File: pcb/pcb.kicad_pcb (KiCad board)
At the start: 2 copper layers, 272.3 x 77.6 mm, 134 parts, among them J1 USB_C_Receptacle_USB2.0, J2 AVR-ISP-6, SW1 SW_Push, U1 ATmega32U4-AU, U2 PRTR5V0U2X, Y1 16MHz

Commit message: create readme
Parts:
- removed G1: LOGO, graphics:logo.pretty
- renumbered D51 to LED1
